Commit message: robot adde to an environment + direct teleop works

File: src/mecanum_robot_description/urdf/urdf/imu.urdf.xacro (robot description, xacro)
@@ -62,8 +62,8 @@
             </material>
             <sensor name="${prefix}imu_sensor" type="imu">
-                <topic>imu</topic>
+                <topic>${topic_name}</topic>
                 <update_rate>${update_rate}</update_rate>
                 <always_on>${always_on}</always_on>
-                <visualize>true</visualize>
+                <visualize>${visualize}</visualize>
                 <gz_frame_id>${prefix}${frame_id}_link</gz_frame_id>
             </sensor>

File: src/mecanum_robot_description/urdf/urdf/lidar.urdf.xacro (robot description, xacro)
@@ -81,5 +81,5 @@
         <specular>${gazebo_material_specular}</specular>
       </material>
-      <sensor name="${prefix}lidar_sensor" type="gpu_lidar">
+      <sensor name="${prefix}${frame_id}_sensor" type="lidar">
         <topic>${topic_name}</topic>
         <update_rate>${update_rate}</update_rate>

File: src/mecanum_robot_description/urdf/urdf/lift.urdf.xacro (robot description, xacro)
@@ -2,5 +2,5 @@
 <robot xmlns:xacro="http://www.ros.org/wiki/xacro">
   <xacro:property name="lift_mass" value="5.0" />
-  <xacro:property name="lift_range" value="0.5" />
+  <xacro:property name="lift_range" value="0.25" />
   <xacro:macro name="lift_mechanism" params="prefix parent_link">
     <link name="${prefix}lift_link">
@@ -27,9 +27,14 @@
     </link>
     <joint name="${prefix}lift_joint" type="prismatic">
-      <parent link="${parent_link}"/>
+      <parent link="${prefix}${parent_link}"/>
       <child link="${prefix}lift_link"/>
       <origin xyz="0 0 0.15" rpy="0 0 0"/>
       <axis xyz="0 0 1"/>
-      <limit lower="0" upper="${lift_range}" effort="200" velocity="0.2"/>
+      <limit lower="0" upper="${lift_range}" effort="200" velocity="0.12"/>
+      <safety_controller
+        soft_lower_limit="0.0"
+        soft_upper_limit="${lift_range}"
+        k_position="50.0"
+        k_velocity="20.0"/>
       <dynamics damping="15.0" friction="2.0"/>
     </joint>
@@ -45,4 +50,14 @@
     <gazebo reference="${prefix}lift_link">
       <material>Gazebo/Grey</material>
+      <collision>
+        <surface>
+          <friction>
+            <ode>
+              <mu>10.0</mu>
+              <mu2>10.0</mu2>
+            </ode>
+          </friction>
+        </surface>
+      </collision>
     </gazebo>
   </xacro:macro>

File: src/mecanum_robot_description/urdf/urdf/robot.urdf.xacro (robot description, xacro)
@@ -11,5 +11,7 @@
     <xacro:include filename="$(find mecanum_robot_description)/urdf/urdf/materials.xacro"/>
     <xacro:include filename="$(find mecanum_robot_description)/urdf/urdf/lift.urdf.xacro"/>
-    <xacro:include filename="$(find mecanum_robot_description)/urdf/plugins/mecanum_robot.gazebo"/>
+    <xacro:if value="$(arg use_gazebo)">
+      <xacro:include filename="$(find mecanum_robot_description)/urdf/plugins/mecanum_robot.gazebo"/>
+    </xacro:if>
     <!-- base -->
     <xacro:base prefix="$(arg prefix)"/>
@@ -76,5 +78,6 @@
       topic_name="imu/data"/>
     <!-- Add Gazebo frictions -->
-    <gazebo reference='front_left_wheel_link'>
+    <xacro:if value="$(arg use_gazebo)">
+    <gazebo reference='$(arg prefix)front_left_wheel_link'>
       <collision>
         <surface>
@@ -83,5 +86,5 @@
               <mu>8</mu>
               <mu2>0.0</mu2>
-              <fdir1 gz:expressed_in="base_footprint">1 -1 0</fdir1>
+              <fdir1 gz:expressed_in="$(arg prefix)base_footprint">1 -1 0</fdir1>
             </ode>
           </friction>
@@ -89,5 +92,5 @@
       </collision>
     </gazebo>
-    <gazebo reference='back_left_wheel_link'>
+    <gazebo reference='$(arg prefix)back_left_wheel_link'>
       <collision>
         <surface>
@@ -96,5 +99,5 @@
               <mu>8</mu>
               <mu2>0.0</mu2>
-              <fdir1 gz:expressed_in="base_footprint">1 1 0</fdir1>
+              <fdir1 gz:expressed_in="$(arg prefix)base_footprint">1 1 0</fdir1>
             </ode>
           </friction>
@@ -102,5 +105,5 @@
       </collision>
     </gazebo>
-    <gazebo reference='front_right_wheel_link'>
+    <gazebo reference='$(arg prefix)front_right_wheel_link'>
       <collision>
         <surface>
@@ -109,5 +112,5 @@
               <mu>8</mu>
               <mu2>0.0</mu2>
-              <fdir1 gz:expressed_in="base_footprint">1 1 0</fdir1>
+              <fdir1 gz:expressed_in="$(arg prefix)base_footprint">1 1 0</fdir1>
             </ode>
           </friction>
@@ -115,5 +118,5 @@
       </collision>
     </gazebo>
-    <gazebo reference='back_right_wheel_link'>
+    <gazebo reference='$(arg prefix)back_right_wheel_link'>
       <collision>
         <surface>
@@ -122,5 +125,5 @@
               <mu>8</mu>
               <mu2>0.0</mu2>
-              <fdir1 gz:expressed_in="base_footprint">1 -1 0</fdir1>
+              <fdir1 gz:expressed_in="$(arg prefix)base_footprint">1 -1 0</fdir1>
             </ode>
           </friction>
@@ -128,7 +131,8 @@
       </collision>
     </gazebo>
-    <gazebo reference="base_link">
+    <gazebo reference="$(arg prefix)base_link">
       <mu1>0.000002</mu1>
       <mu2>0.000002</mu2>
     </gazebo>
+    </xacro:if>
 </robot>
